File: sQrt_niu_heimar.kicad_pcb (KiCad board)
At the start: 2 copper layers, 84 x 100 mm, 130 parts, among them J1 NMJ6HCD2, J2 NMJ6HCD2, J3 MJ-179PH, Q1 2SC2240, Q2 2SK303, Q3 2SK303, SW1 SW_SPST, U1 TL074, U2 TL074, U4 MC34063AP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

Commit message: v1.0.1_test
Parts:
- moved R42 0.10 mm to (229.0, 42.5)
Changed lines of the file:
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@@
   )
   (footprint "Resistor_THT:R_Axial_DIN0207_L6.3mm_D2.5mm_P7.62mm_Horizontal" (layer "F.Cu")
-    (at 228.97 42.6)
+    (at 228.97 42.5)
     (descr "Resistor, Axial_DIN0207 series, Axial, Horizontal, pin pitch=7.62mm, 0.25W = 1/4W, length*diameter=6.3*2.5mm^2, http://cdn-reichelt.de/documents/datenblatt/B400/1_4W%23YAG.pdf")
     (tags "Resistor Axial_DIN0207 series Axial Horizontal pin pitch 7.62mm 0.25W = 1/4W length 6.3mm diameter 2.5mm")

Commit message: v2.0.0
Parts:
- C29, C30, C31, C32: footprint Capacitor_THT:C_Rect_L7.2mm_W5.5mm_P5.00mm_FKS2_FKP2_MKS2_MKP2 -> Capacitor_THT:C_Rect_L7.2mm_W2.5mm_P5.00mm_FKS2_FKP2_MKS2_MKP2
- C3: footprint Capacitor_THT:C_Rect_L8.5mm_W5.5mm_P5.00mm_FKS2_FKP2_MKS2_MKP2 -> Capacitor_THT:C_Rect_L7.2mm_W2.5mm_P5.00mm_FKS2_FKP2_MKS2_MKP2
- L1: footprint Inductor_THT:L_Axial_L14.0mm_D4.5mm_P15.24mm_Horizontal_Fastron_LACC -> Inductor_THT:L_Axial_L11.0mm_D4.5mm_P5.08mm_Vertical_Fastron_MECC
- RV1, RV2, RV3, RV4, RV5, RV6, RV7, RV8, RV9: moved to B.Cu
- moved C24 171.7 mm to (107.5, 138.7)
- moved C7 154.2 mm to (131.7, 129.0)
- moved C30 143.9 mm to (138.2, 139.7), turned to 180 degrees
- moved C31 141.9 mm to (133.4, 136.8), turned to 90 degrees
- moved C9 141.1 mm to (132.0, 107.2)
- moved R66 139.6 mm to (105.0, 99.3), turned to 90 degrees
- moved R64 139.1 mm to (105.0, 89.6), turned to 90 degrees
- moved R46 139.1 mm to (113.0, 135.6)
- moved R41 137.7 mm to (128.3, 132.6), turned to 180 degrees
- moved R67 135.6 mm to (108.0, 99.3), turned to 90 degrees
- moved C32 135.5 mm to (136.4, 136.8), turned to 90 degrees
- moved R65 135.3 mm to (108.0, 89.6), turned to 90 degrees
- moved C29 134.7 mm to (151.7, 134.3), turned to -90 degrees
- moved C17 133.7 mm to (127.6, 69.0), turned to 90 degrees
- moved C11 133.3 mm to (124.0, 77.2), turned to 90 degrees
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Connections:
- R49 pad 1: -5v -> -7.3V
- R50 pad 1: -5v -> -7.3V
- R52 pad 2: Net-(R14-Pad1) -> Net-(R52-Pad2)
- R58 pad 1: Net-(U1A--) -> Net-(R52-Pad2)
- R59 pad 2: Net-(R13-Pad1) -> Net-(R59-Pad2)
- R61 pad 1: Net-(C4-Pad1) -> Net-(R59-Pad2)
- R62 pad 1: Net-(C12-Pad1) -> Net-(R62-Pad1)
- R63 pad 2: Net-(R22-Pad1) -> Net-(R62-Pad1)
- R64 pad 1: Net-(C16-Pad1) -> Net-(R64-Pad1)
- R65 pad 2: Net-(R32-Pad1) -> Net-(R64-Pad1)
- R66 pad 2: Net-(R33-Pad1) -> Net-(R66-Pad2)
- R67 pad 1: Net-(U2C--) -> Net-(R66-Pad2)
- R68 pad 2: Net-(R23-Pad1) -> Net-(R68-Pad2)
- R69 pad 1: Net-(U2A--) -> Net-(R68-Pad2)
- U7 pad 6: -5v -> -7.3V
- U7 pad 7: -5v -> -7.3V
Routing:
- net 7.3V: track 67.1 -> 317.9 mm, vias 0 -> 3
- net -7.3V: track 78.1 -> 279.7 mm
- net Net-(U7A-D): track 0.00 -> 136.3 mm, vias 0 -> 1
- net Net-(Q1-B): track 0.00 -> 135.8 mm, vias 0 -> 3
- net Net-(Q2-S): track 0.00 -> 130.3 mm, vias 0 -> 3
- net GND: track 0.00 -> 114.3 mm, vias 0 -> 6
- net Net-(U1A--): track 0.00 -> 110.9 mm, vias 0 -> 4
- net Net-(C4-Pad1): track 0.00 -> 109.3 mm, vias 0 -> 3
- net Net-(C16-Pad1): track 0.00 -> 106.1 mm, vias 0 -> 2
- net Net-(U2C--): track 0.00 -> 101.2 mm, vias 0 -> 2
- net Net-(U1B--): track 0.00 -> 100.5 mm, vias 0 -> 2
- net Net-(C7-Pad2): track 0.00 -> 98.7 mm, vias 0 -> 2
- net Net-(Q2-D): track 0.00 -> 96.4 mm, vias 0 -> 2
- net Net-(U5A--): track 0.00 -> 94.9 mm, vias 0 -> 3
- net Net-(U1C--): track 0.00 -> 92.8 mm, vias 0 -> 2
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- added copper zone on B.Cu, net GND
- added copper zone on F.Cu, net GND
