File: sQrt_niu_heimar.kicad_sch (KiCad schematic)
At the start: 130 parts, among them J1 NMJ6HCD2, J2 NMJ6HCD2, J3 MJ-179PH, Q1 2SC2240, Q2 2SK303, Q3 2SK303, SW1 SW_SPST, U1 TL074, U2 TL074, U4 MC34063AP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

Commit message: v1.0.1_test
Other:
- moved on the sheet: R42
Changed lines of the file:
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@@
     (stroke (width 0) (type default))
   )
-  (wire (pts (xy 203.2 31.75) (xy 207.01 31.75))
+  (wire (pts (xy 203.2 30.48) (xy 207.01 30.48))
     (stroke (width 0) (type default))
   )
@@
     (stroke (width 0) (type default))
   )
-  (wire (pts (xy 222.25 31.75) (xy 222.25 41.91))
+  (wire (pts (xy 222.25 30.48) (xy 222.25 41.91))
     (stroke (width 0) (type default))
   )
@@
     (stroke (width 0) (type default))
   )
-  (wire (pts (xy 203.2 31.75) (xy 203.2 41.91))
+  (wire (pts (xy 203.2 30.48) (xy 203.2 41.91))
     (stroke (width 0) (type default))
   )
@@
     (stroke (width 0) (type default))
   )
-  (wire (pts (xy 214.63 31.75) (xy 222.25 31.75))
+  (wire (pts (xy 214.63 30.48) (xy 222.25 30.48))
     (stroke (width 0) (type default))
   )
@@
     )
   )
-  (symbol (lib_id "Device:R") (at 210.82 31.75 90) (unit 1)
-    (in_bom yes) (on_board yes) (dnp no) (fields_autoplaced)
-    (property "Reference" "R42" (at 210.82 25.4 90)
-      (effects (font (size 1.27 1.27)))
-    )
-    (property "Value" "10k" (at 210.82 27.94 90)
-      (effects (font (size 1.27 1.27)))
-    )
-    (property "Footprint" "Resistor_THT:R_Axial_DIN0207_L6.3mm_D2.5mm_P7.62mm_Horizontal" (at 210.82 33.528 90)
-      (effects (font (size 1.27 1.27)) hide)
-    )
-    (property "Datasheet" "~" (at 210.82 31.75 0)
-      (effects (font (size 1.27 1.27)) hide)
-    )
+  (symbol (lib_id "Device:R") (at 210.82 30.48 90) (unit 1)
+    (in_bom yes) (on_board yes) (dnp no) (fields_autoplaced)
+    (property "Reference" "R42" (at 210.82 24.13 90)
+      (effects (font (size 1.27 1.27)))
+    )
+    (property "Value" "10k" (at 210.82 26.67 90)
+      (effects (font (size 1.27 1.27)))
+    )
+    (property "Footprint" "Resistor_THT:R_Axial_DIN0207_L6.3mm_D2.5mm_P7.62mm_Horizontal" (at 210.82 32.258 90)
+      (effects (font (size 1.27 1.27)) hide)
+    )
+    (property "Datasheet" "~" (at 210.82 30.48 0)
+      (effects (font (size 1.27 1.27)) hide)
+    )

Commit message: v2.0.0
Parts:
- C29, C30, C31, C32: footprint Capacitor_THT:C_Rect_L7.2mm_W5.5mm_P5.00mm_FKS2_FKP2_MKS2_MKP2 -> Capacitor_THT:C_Rect_L7.2mm_W2.5mm_P5.00mm_FKS2_FKP2_MKS2_MKP2
- C3: footprint Capacitor_THT:C_Rect_L8.5mm_W5.5mm_P5.00mm_FKS2_FKP2_MKS2_MKP2 -> Capacitor_THT:C_Rect_L7.2mm_W2.5mm_P5.00mm_FKS2_FKP2_MKS2_MKP2
- L1: footprint Inductor_THT:L_Axial_L14.0mm_D4.5mm_P15.24mm_Horizontal_Fastron_LACC -> Inductor_THT:L_Axial_L11.0mm_D4.5mm_P5.08mm_Vertical_Fastron_MECC
Connections:
- net -5v is gone; now on net -7.3V: R49.1, R50.1, U7.6 (S), U7.7 (VSS)
- net at C12.1, R24.1, R63.1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: no longer R62.1
- net at R22.1, R62.2, RV8.1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: no longer R63.2
- net at R14.1, R58.2, RV7.4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: no longer R52.2
- net at C4.2, C8.2, R52.1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: no longer R58.1
- net at C16.1, C17.1, R34.1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: no longer R64.1
- net at C16.2, C17.2, R66.1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: no longer R67.1
- net at C12.2, R68.1, RV8.6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: no longer R69.1
- net at R13.1, R61.2, RV7.1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: no longer R59.2
- net at C4.1, C8.1, R15.1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: no longer R61.1
- net at R32.1, R64.2, RV9.1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: no longer R65.2
- net at R33.1, R67.2, RV9.4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: no longer R66.2
- net at R23.1, R69.2, RV8.4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: no longer R68.2
- new net: R62.1, R63.2
- new net: R52.2, R58.1
- new net: R66.2, R67.1
- new net: R68.2, R69.1
- new net: R64.1, R65.2
- new net: R59.2, R61.1
Other:
- moved on the sheet: C15, C19, C20, C28, C35, D4, L1, R51, R53, RV10, U4
